Commit message: adding teleop and more bite objects

File: assistive_gym/envs/assets/food_items/strawberry.urdf (robot description, URDF)
Before this commit: robot strawberry.urdf, 1 links, 0 joints
Links:
- link base: mass 0.012 -> 0.002

File: assistive_gym/envs/assets/mouth/hole.urdf (robot description, URDF)
Before this commit: robot hole.urdf, 1 links, 0 joints
Links:
- link base: geometry collision mesh filename=hole2_vhacd.obj scale=0.035 0.035 0.06; visual mesh filename=hole2.obj scale=0.035 0.035 0.06
